File: WiFi-Gate-Control-Board-Inputs.sch (KiCad schematic (older format))
At the start: 112 parts, among them J4 Screw_Terminal_01x04, J5 Screw_Terminal_01x04, J6 Screw_Terminal_01x04, J7 Screw_Terminal_01x04, J8 Screw_Terminal_01x04, J9 Screw_Terminal_01x04, SW1 LED Enable, SW2 Open-Close, U10 TPS3779, U11 TPS3779, U12 TPS3779, U13 TPS3779, U14 TCA6424A, U15 REF3330, U16 TPS3779, U17 TPS3779, U18 TPS3779, U19 TPS3779, U20 TPS3779, U21 TPS3779, U22 TPS3779, U23 TPS3779

Commit message: Rev 1.0 Release
Added input design and calculations. Added BOM. Added Fuse 3D Model.
Parts:
- D10: renamed from D11; Description IC, SOT-23, Dual ESD Protection Device -> TVS, SC70-3, ESD TVS Protection, Dual; Part Number TPD2E2U06QDBZRQ1 -> TPD2E2U06QDCKRQ1; Vendor Part Number 595-TPD2E2U06QDBZRQ1 -> 595-TPD2E2U06QDCKRQ1
- D11: renamed from D12; Description IC, SOT-23, Dual ESD Protection Device -> TVS, SC70-3, ESD TVS Protection, Dual; Part Number TPD2E2U06QDBZRQ1 -> TPD2E2U06QDCKRQ1; Vendor Part Number 595-TPD2E2U06QDBZRQ1 -> 595-TPD2E2U06QDCKRQ1
- D12: renamed from D13; Description IC, SOT-23, Dual ESD Protection Device -> TVS, SC70-3, ESD TVS Protection, Dual; Part Number TPD2E2U06QDBZRQ1 -> TPD2E2U06QDCKRQ1; Vendor Part Number 595-TPD2E2U06QDBZRQ1 -> 595-TPD2E2U06QDCKRQ1
- D7: renamed from D8; Description IC, SOT-23, Dual ESD Protection Device -> TVS, SC70-3, ESD TVS Protection, Dual; Part Number TPD2E2U06QDBZRQ1 -> TPD2E2U06QDCKRQ1; Vendor Part Number 595-TPD2E2U06QDBZRQ1 -> 595-TPD2E2U06QDCKRQ1
- D8: renamed from D9; Description IC, SOT-23, Dual ESD Protection Device -> TVS, SC70-3, ESD TVS Protection, Dual; Part Number TPD2E2U06QDBZRQ1 -> TPD2E2U06QDCKRQ1; Vendor Part Number 595-TPD2E2U06QDBZRQ1 -> 595-TPD2E2U06QDCKRQ1
- D9: renamed from D10; Description IC, SOT-23, Dual ESD Protection Device -> TVS, SC70-3, ESD TVS Protection, Dual; Part Number TPD2E2U06QDBZRQ1 -> TPD2E2U06QDCKRQ1; Vendor Part Number 595-TPD2E2U06QDBZRQ1 -> 595-TPD2E2U06QDCKRQ1
- renumbered C42 to C25, C43 to C26, C44 to C27, C45 to C28, C46 to C29, C47 to C30, C48 to C31, C49 to C32, C50 to C33, C51 to C34, C52 to C35, C53 to C36, C54 to C37, C55 to C38, C56 to C39, C57 to C40, C58 to C41, C59 to C42, C60 to C43, C61 to C44, C62 to C45, C63 to C46, C64 to C47, C65 to C48, C66 to C49, C67 to C50, C68 to C51, C69 to C52, C70 to C53, F2 to F1, F3 to F2, J4 to J3, J5 to J4, J6 to J5, J7 to J6, J8 to J7, J9 to J8, R22 to R10, R23 to R11, R24 to R12, R25 to R13, R26 to R14, R27 to R15, R28 to R16, R29 to R17, R30 to R18, R31 to R19, R32 to R20, R33 to R21, R34 to R22, R35 to R23, R36 to R24, R37 to R25, R38 to R26, R39 to R27, R40 to R28, R41 to R29, R42 to R30, R43 to R31, R44 to R32, R45 to R33, R46 to R34, R47 to R35, R48 to R36, R49 to R37, R50 to R38, R51 to R39, R52 to R40, R53 to R41, R54 to R42, R55 to R43, R56 to R44, R57 to R45, R58 to R46, R59 to R47, R60 to R48, R61 to R49, R62 to R50, R63 to R51, R64 to R52, R65 to R53, R66 to R54, R67 to R55, R68 to R56, R69 to R57, R70 to R58, R71 to R59, R72 to R60, R73 to R61, R74 to R62, U13 to U10, U14 to U11, U15 to U12, U16 to U13, U17 to U14, U18 to U15, U19 to U16, U20 to U17, U21 to U18, U22 to U19, U23 to U20, U10 to U7, U11 to U8, U12 to U9

Commit message: PCB to Rev 1.1
Fixed missing Reference Designators on top Silkscreen.
Reset input on TCA6424A and TCA6408A now connected to 3.3V.
Added series Schottky Diode to LED power supply input.
Replaced 1000uF main power capacitor with two 470uF capacitors.
Replaced DS18B20 temperature sensor with TMP100 temperature sensor.
Increased LED currents to 25mA
Removed U26 inverter and connected U3 IN pin directly to processor. Now able to measure unloaded offset current.
Parts:
- added TP3: SDA, TestPoint:TestPoint_THTPad_D1.5mm_Drill0.7mm, symbol Connector:TestPoint
- added TP4: SCL, TestPoint:TestPoint_THTPad_D1.5mm_Drill0.7mm, symbol Connector:TestPoint
- J3, J4, J5, J6, J7, J8: value Screw_Terminal_01x04 -> Screw Header 4 Pos; Description CON, THT, 5.08mm Pluggable Terminal Strip, 4 Pos -> CON, THT, 5.08mm Pluggable Terminal Header, 4 Pos
- R10: renamed from R11; Description RES, 0603, 6.81k, 1/16W, 0.5%, T25 -> RES, 0603, 33.2k, 1/16W, 0.5%, T25
- R20: renamed from R21; Description RES, 0603, 6.81k, 1/16W, 0.5%, T25 -> RES, 0603, 33.2k, 1/16W, 0.5%, T25
- R21: renamed from R22; Description RES, 0603, 6.81k, 1/16W, 0.5%, T25 -> RES, 0603, 33.2k, 1/16W, 0.5%, T25
- R28: renamed from R29; Description RES, 0603, 6.81k, 1/16W, 0.5%, T25 -> RES, 0603, 33.2k, 1/16W, 0.5%, T25
- R29: renamed from R30; Description RES, 0603, 6.81k, 1/16W, 0.5%, T25 -> RES, 0603, 33.2k, 1/16W, 0.5%, T25
- R36: renamed from R37; Description RES, 0603, 6.81k, 1/16W, 0.5%, T25 -> RES, 0603, 33.2k, 1/16W, 0.5%, T25
- R37: renamed from R38; Description RES, 0603, 6.81k, 1/16W, 0.5%, T25 -> RES, 0603, 33.2k, 1/16W, 0.5%, T25
- R46: renamed from R47; Description RES, 0603, 6.81k, 1/16W, 0.5%, T25 -> RES, 0603, 33.2k, 1/16W, 0.5%, T25
- R47: renamed from R48; Description RES, 0603, 6.81k, 1/16W, 0.5%, T25 -> RES, 0603, 33.2k, 1/16W, 0.5%, T25
- R54: renamed from R55; Description RES, 0603, 6.81k, 1/16W, 0.5%, T25 -> RES, 0603, 33.2k, 1/16W, 0.5%, T25
- R55: renamed from R56; Description RES, 0603, 6.81k, 1/16W, 0.5%, T25 -> RES, 0603, 33.2k, 1/16W, 0.5%, T25
- R9: renamed from R10; Description RES, 0603, 6.81k, 1/16W, 0.5%, T25 -> RES, 0603, 33.2k, 1/16W, 0.5%, T25
- SW1: value LED Enable -> ~
- SW2: value Open-Close -> ~
- renumbered R12 to R11, R13 to R12, R14 to R13, R15 to R14, R16 to R15, R17 to R16, R18 to R17, R19 to R18, R20 to R19, R23 to R22, R24 to R23, R25 to R24, R26 to R25, R27 to R26, R28 to R27, R31 to R30, R32 to R31, R33 to R32, R34 to R33, R35 to R34, R36 to R35, R39 to R38, R40 to R39, R41 to R40, R42 to R41, R43 to R42, R44 to R43, R45 to R44, R46 to R45, R49 to R48, R50 to R49, R51 to R50, R52 to R51, R53 to R52, R54 to R53, R57 to R56, R58 to R57, R59 to R58, R60 to R59, R61 to R60, R62 to R61
Connections:
- net +3.3V: now also U11.28 (~RESET)
- net SCL: now also TP4.1
- net SDA: now also TP3.1
Other:
- note added: "Address 010 0010"
- note added: "LED Enable"
- note added: "Open-Close"
- note removed: "Address 010 0010."
