File: WiFi-Gate-Control-Board-Motor.sch (KiCad schematic (older format))
At the start: 40 parts, among them J3 Motor, Q1 IPD90P03P4L-04, Q2 IFX007T, Q3 IFX007T, U7 74LVC2G17, U8 74LVC1G04, U9 REF3325

Commit message: Rev 1.0 Release
Added input design and calculations. Added BOM. Added Fuse 3D Model.
Parts:
- C67: renamed from C28; Manufacturer Microchip -> Taiyo Yuden
- C68: renamed from C29; Manufacturer Microchip -> Taiyo Yuden
- C71: renamed from C32; Manufacturer Microchip -> Taiyo Yuden
- C72: renamed from C33; Manufacturer Microchip -> Taiyo Yuden
- D28: renamed from D7; footprint Package_TO_SOT_SMD:SOT-23 -> Package_TO_SOT_SMD:SOT-323_SC-70; Description TVS, SOT23, ESD TVS Protection, Dual -> TVS, SC70-3, ESD TVS Protection, Dual; Part Number TPD2E2U06QDBZRQ1 -> TPD2E2U06QDCKRQ1; Vendor Part Number 595-TPD2E2U06QDBZRQ1 -> 595-TPD2E2U06QDCKRQ1
- Z1: footprint Diode_SMD:D_SOD-523 -> Diode_SMD:D_SOT-23_ANK; Description Zener, 10V, SOD523 -> Zener, 10V, SOT-23; Manufacturer Diodes Inc -> On Semiconductor; Part Number DDZ9697T-7 -> SZBZX84C10LT1G; Vendor Part Number 621-DDZ9697T-7 -> 863-SZBZX84C10LT1G
- renumbered C25 to C64, C26 to C65, C27 to C66, C30 to C69, C31 to C70, C34 to C73, C35 to C74, C36 to C75, C37 to C76, C38 to C77, C39 to C78, C40 to C79, C41 to C80, F1 to F3, J3 to J12, R10 to R75, R11 to R76, R12 to R77, R13 to R78, R14 to R79, R15 to R80, R16 to R81, R17 to R82, R18 to R83, R19 to R84, R20 to R85, R21 to R86, U7 to U25, U8 to U26, U9 to U27

Commit message: PCB to Rev 1.1
Fixed missing Reference Designators on top Silkscreen.
Reset input on TCA6424A and TCA6408A now connected to 3.3V.
Added series Schottky Diode to LED power supply input.
Replaced 1000uF main power capacitor with two 470uF capacitors.
Replaced DS18B20 temperature sensor with TMP100 temperature sensor.
Increased LED currents to 25mA
Removed U26 inverter and connected U3 IN pin directly to processor. Now able to measure unloaded offset current.
Parts:
- removed C77: 0.1uF, Capacitor_SMD:C_0603_1608Metric, symbol Device:C
- removed R86: 10k, Resistor_SMD:R_0603_1608Metric, symbol Device:R
- removed U26: 74LVC1G04, Package_TO_SOT_SMD:SOT-23-5, symbol 74xGxx:74LVC1G04
- added C65: 470uF, Capacitor_THT:CP_Radial_D16.0mm_P7.50mm, symbol Device:CP1
- added C67, C68: DNI, Capacitor_SMD:C_0603_1608Metric, symbol Device:C
- added R80: 10k, Resistor_SMD:R_0603_1608Metric, symbol Device:R
- C66: renamed from C65; value 1000uF -> 470uF; Description CAP, THT 16X20, 1000uF, 20%, EC, 35V -> CAP, THT 16X15, 470uF, 20%, EC, 35V; Manufacturer Panasonic -> Nichicon; Part Number EEU-FC1V102S -> UPM1V471MHD6; Tolerance (none) -> 20%; Vendor Part Number 667-EEU-FC1V102S -> 647-UPM1V471MHD6
- Q1: Vendor Part Number 849-CPC1511 -> 726-IPD90P03P4L04
- R74: renamed from R75; Vendor Part Number 667-ERJ-P08J104V -> 667-ERJ-P08J334V
- R75: renamed from R76; Vendor Part Number 667-ERJ-P08J104V -> 667-ERJ-P08J334V
- R76: renamed from R77; Description RES, 0603, 10k, 1/10W, 1%, T100 -> RES, 0603, 10k, 1/16W, 0.5%, T25; Manufacturer Panasonic -> Susumu; Part Number ERJ-3EKF1002V -> RR0816P-103-D; Tolerance 1% -> 0.5%; Vendor Part Number 667-ERJ-3EKF1002V -> 754-RR0816P-103D
- R79: renamed from R80; Description RES, 0603, 10k, 1/10W, 1%, T100 -> RES, 0603, 10k, 1/16W, 0.5%, T25; Manufacturer Panasonic -> Susumu; Part Number ERJ-3EKF1002V -> RR0816P-103-D; Tolerance 1% -> 0.5%; Vendor Part Number 667-ERJ-3EKF1002V -> 754-RR0816P-103D
- R81, R84, R85: Description RES, 0603, 10k, 1/10W, 1%, T100 -> RES, 0603, 10k, 1/16W, 0.5%, T25; Manufacturer Panasonic -> Susumu; Part Number ERJ-3EKF1002V -> RR0816P-103-D; Tolerance 1% -> 0.5%; Vendor Part Number 667-ERJ-3EKF1002V -> 754-RR0816P-103D
- renumbered C66 to C69, C67 to C70, C68 to C71, C69 to C72, C70 to C73, C71 to C74, C72 to C75, C73 to C76, C74 to C77, C75 to C78, C76 to C79, C78 to C80, C79 to C81, C80 to C82, D28 to D29, R78 to R77, R79 to R78, U27 to U26
Connections:
- net +12V: now also C65.1
- net GND: now also C65.2, C67.2, C68.1
- net at Q3.2 (IN): now also R80.1
- net at D29.1 (IO1), R77.2, U25.1: now also C67.1
- net at D29.2 (IO2), R78.2, U25.3: now also C68.2
- new net A5: R80.2
Other:
- note added: "MEXTH"
- note added: "MEXTL"
- note added: "Offset Measurement (Motor Off)"
- note added: "Unused (Motor Off)"
- note removed: "MEXT"
- moved on the sheet: C66, F3, Q1, R74, R75, R76, R77, R78, Z1
