File: WiFi-Gate-Control-Board.sch (KiCad schematic (older format))
At the start: 52 parts, among them J1 USB_B_Micro, J2 Cortex Debug, U1 LMZ21700, U2 DS18B20U, U3 ATWINC1500-MR210UB, U4 SAMD21G18-M, U5 74LVC2G07, U6 74LVC2G06, Y1 32.768kHz

Commit message: Rev 1.0 Release
Added input design and calculations. Added BOM. Added Fuse 3D Model.
Parts:
- C2, C3, C4, C5: Description CAP, 0603, 1000pF, 10%, X7R, 10V -> CAP, 0603, 1nF, 10%, X7R, 10V
- C8: Description CAP, 0603, 3300pF, 5%, X7R, 10V -> CAP, 0603, 3.3nF, 5%, X7R, 10V
- D3: Description TVS, SOT23, ESD Protection, USB -> TVS, SOT143, ESD Protection, USB
Other:
- note removed: "3."
- note removed: "All LEDs are normally off."
Changed lines of the file:
@@
 F 8 "50V" H 2600 2200 50  0000 L CNN "Voltage"
 F 9 "10%" H 2500 2100 60  0001 C CNN "Tolerance"
-F 10 "CAP, 0603, 1000pF, 10%, X7R, 10V" H 2500 2100 50  0001 C CNN "Description"
+F 10 "CAP, 0603, 1nF, 10%, X7R, 10V" H 2500 2100 50  0001 C CNN "Description"
 	1    2500 2100
 	-1   0    0    1
@@
 F 8 "50V" H 3100 2200 50  0000 L CNN "Voltage"
 F 9 "10%" H 3000 2100 60  0001 C CNN "Tolerance"
-F 10 "CAP, 0603, 1000pF, 10%, X7R, 10V" H 3000 2100 50  0001 C CNN "Description"
+F 10 "CAP, 0603, 1nF, 10%, X7R, 10V" H 3000 2100 50  0001 C CNN "Description"
 	1    3000 2100
 	1    0    0    1
@@
 F 8 "50V" H 1650 2200 50  0000 L CNN "Voltage"
 F 9 "10%" H 1550 2100 60  0001 C CNN "Tolerance"
-F 10 "CAP, 0603, 1000pF, 10%, X7R, 10V" H 1550 2100 50  0001 C CNN "Description"
+F 10 "CAP, 0603, 1nF, 10%, X7R, 10V" H 1550 2100 50  0001 C CNN "Description"
 	1    1550 2100
 	-1   0    0    1
@@
 F 6 "Mouser" H 2450 6000 50  0001 C CNN "Vendor"
 F 7 "771-PRTR5V0U2X-T/R" H 2450 6000 50  0001 C CNN "Vendor Part Number"
-F 8 "TVS, SOT23, ESD Protection, USB" H 2450 6000 50  0001 C CNN "Description"
+F 8 "TVS, SOT143, ESD Protection, USB" H 2450 6000 50  0001 C CNN "Description"
 	1    2450 6000
 	1    0    0    -1
@@
 F 8 "50V" H 2150 2200 50  0000 L CNN "Voltage"
 F 9 "10%" H 2050 2100 60  0001 C CNN "Tolerance"
-F 10 "CAP, 0603, 1000pF, 10%, X7R, 10V" H 2050 2100 50  0001 C CNN "Description"
+F 10 "CAP, 0603, 1nF, 10%, X7R, 10V" H 2050 2100 50  0001 C CNN "Description"
 	1    2050 2100
 	-1   0    0    1
@@
 F 8 "10V" H 4550 2000 50  0000 L CNN "Voltage"
 F 9 "5%" H 4450 2100 60  0001 C CNN "Tolerance"
-F 10 "CAP, 0603, 3300pF, 5%, X7R, 10V" H 4450 2100 50  0001 C CNN "Description"
+F 10 "CAP, 0603, 3.3nF, 5%, X7R, 10V" H 4450 2100 50  0001 C CNN "Description"
 	1    4450 2100
 	-1   0    0    -1
@@
 Text Notes 650  9250 0    150  ~ 0
 Notes
-Text Notes 650  9900 0    100  Italic 0
-3.
-Text Notes 850  9900 0    100  Italic 0
-All LEDs are normally off.
 Wire Bus Line
 	6900 4050 6900 8950

Commit message: PCB to Rev 1.1
Fixed missing Reference Designators on top Silkscreen.
Reset input on TCA6424A and TCA6408A now connected to 3.3V.
Added series Schottky Diode to LED power supply input.
Replaced 1000uF main power capacitor with two 470uF capacitors.
Replaced DS18B20 temperature sensor with TMP100 temperature sensor.
Increased LED currents to 25mA
Removed U26 inverter and connected U3 IN pin directly to processor. Now able to measure unloaded offset current.
Parts:
- removed R1: 4.7k, Resistor_SMD:R_0603_1608Metric, symbol Device:R
- removed U2: DS18B20U, Package_SO:MSOP-8_3x3mm_P0.65mm, symbol Sensor_Temperature:DS18B20U
- added TP1, TP2: TestPoint_Probe, TestPoint:TestPoint_Pad_D1.0mm, symbol Connector:TestPoint_Probe
- added U2: TMP100, Package_TO_SOT_SMD:SOT-23-6, symbol Sensor_Temperature:TMP100
- R3: renamed from R4; value 143R -> 44.2R; Description RES, 0603, 143R, 1/10W, 1%, T100 -> RES, 0603, 44.2R, 1/10W, 1%, T100; Part Number ERJ-3EKF1430V -> ERJ-3EKF44R2V; Vendor Part Number 667-ERJ-3EKF1430V -> 667-ERJ-3EKF44R2V
- R4: renamed from R5; value 143R -> 44.2R; Description RES, 0603, 143R, 1/10W, 1%, T100 -> RES, 0603, 44.2R, 1/10W, 1%, T100; Part Number ERJ-3EKF1430V -> ERJ-3EKF44R2V; Vendor Part Number 667-ERJ-3EKF1430V -> 667-ERJ-3EKF44R2V
- R6: renamed from R7; value 73.2R -> 44.2R; Description RES, 0603, 73.2R, 1/10W, 1%, T100 -> RES, 0603, 44.2R, 1/10W, 1%, T100; Part Number ERJ-3EKF73R2V -> ERJ-3EKF44R2V; Vendor Part Number 667-ERJ-3EKF73R2V -> 667-ERJ-3EKF44R2V
- R7: renamed from R8; value 73.2R -> 44.2R; Description RES, 0603, 73.2R, 1/10W, 1%, T100 -> RES, 0603, 44.2R, 1/10W, 1%, T100; Part Number ERJ-3EKF73R2V -> ERJ-3EKF44R2V; Vendor Part Number 667-ERJ-3EKF73R2V -> 667-ERJ-3EKF44R2V
- R8: renamed from R9; value 73.2R -> 44.2R; Description RES, 0603, 73.2R, 1/10W, 1%, T100 -> RES, 0603, 44.2R, 1/10W, 1%, T100; Part Number ERJ-3EKF73R2V -> ERJ-3EKF44R2V; Vendor Part Number 667-ERJ-3EKF73R2V -> 667-ERJ-3EKF44R2V
- U6: Description SW, THT, Push Button -> IC, SOT-23-6, Dual Inverter with Open-Drain Outputs
- renumbered C2 to C1, C3 to C2, C4 to C3, C5 to C4, C6 to C5, C7 to C6, C8 to C7, C9 to C8, C1 to C9, R2 to R1, R3 to R2, R6 to R5
Connections:
- net +3.3V: now also U2.4 (V+)
- net A2: now also TP1.1
- net A4: now also TP2.1
- net GND: now also U2.2 (GND), U2.3 (ADD1), U2.5 (ADD0)
- net SCL: now also U2.1 (SCL)
- net SDA: now also U2.6 (SDA)
Other:
- note added: "Address 100 1000"
- note added: "MEXTH"
- note added: "MEXTL"
- note added: "Motor Extend High"
- note added: "Motor Extend Low"
- note removed: "1-Wire"
- note removed: "MEXT"
- note removed: "Motor Extend"
- note removed: "OWIRE"
- moved on the sheet: C9

Commit message: Changed Cortex Debug connector. Added fabrication pdf.
Parts:
- J2: Manufacturer Amphenol FCI -> Samtec; Part Number 202112100010C4LF -> FTSH-105-01-L-DV-K; Vendor Part Number 649-202112100010C4LF -> 200-FTSH10501LDVK
Changed lines of the file:
@@
 F 2 "Connector_PinHeader_1.27mm:PinHeader_2x05_P1.27mm_Vertical_SMD" H 2550 7150 50  0001 C CNN
 F 3 "https://www.mouser.com/datasheet/2/18/20021121-1362884.pdf" H 2550 7150 50  0001 C CNN
-F 4 "Amphenol FCI" H 2550 7150 50  0001 C CNN "Manufacturer"
-F 5 "202112100010C4LF" H 2550 7150 50  0001 C CNN "Part Number"
+F 4 "Samtec" H 2550 7150 50  0001 C CNN "Manufacturer"
+F 5 "FTSH-105-01-L-DV-K" H 2550 7150 50  0001 C CNN "Part Number"
 F 6 "Mouser" H 2550 7150 50  0001 C CNN "Vendor"
-F 7 "649-202112100010C4LF" H 2550 7150 50  0001 C CNN "Vendor Part Number"
+F 7 "200-FTSH10501LDVK" H 2550 7150 50  0001 C CNN "Vendor Part Number"
 F 8 "CON, SMD, 1.27mm Header, Dual Row, Vertical, 10 Pos" H 2550 7150 50  0001 C CNN "Description"
 	1    2550 7150
